File: PCB/Control_Pilot.kicad_sch (KiCad schematic)
At the start: 33 parts, among them IC10 TLA431AIDBZR, U4 TLV1805DBVR, U5 TLV1805DBVR

Commit message: Implementação do novo circuito do Wleding detector; correcao dos campos dos componentes
Parts:
- C47, C48: Distribuidor Mouser -> (none); Link https://pt.mouser.com/ProductDetail/Samsung-Electro-Mechani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 -> (none); MPN (none) -> CL10B104MB8NNNC; Ref CL10B104MB8NNNC -> (none)
- C49: Distribuidor Mouser -> (none); Link https://pt.mouser.com/ProductDetail/YAGEO/CC0603JRX7R9BB221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 -> (none); MPN (none) -> CC0603JRX7R9BB221; Ref CC0603JRX7R9BB221 -> (none)
- C50, C51, C53, C54, C55, C57: Distribuidor Mouser -> (none); Link https://pt.mouser.com/ProductDetail/Samsung-Electro-Mechani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 -> (none); MPN (none) -> CL10B105KB8NQNC; Ref CL10B105KB8NQNC -> (none)
- C52: Distribuidor Mouser -> (none); Link https://pt.mouser.com/ProductDetail/KYOCERA-AVX/06035C103MA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 -> (none); MPN (none) -> 06035C103MAZ2A; Ref 06035C103MAZ2A -> (none)
- C56: Distribuidor Mouser -> (none); Link https://pt.mouser.com/ProductDetail/Murata-Electronics/GCM1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 -> (none); MPN (none) -> GCM1885C1H152JA16J; Ref GCM1885C1H152JA16J -> (none)
- D10: Distribuidor Mouser -> (none); Link https://pt.mouser.com/ProductDetail/Vishay-General-Semicond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 -> (none); MPN (none) -> SMAJ14CA-E3/61; Ref SMAJ14CA-E3/61 -> (none)
- D11, D12, D13, D14: Distribuidor Mouser -> (none); Link https://pt.mouser.com/ProductDetail/Diodes-Incorporated/BAT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 -> (none); MPN (none) -> BAT54S-7-F; Ref BAT54S-7-F -> (none)
- IC10: Height 1.12 -> (none); Manufacturer_Name Texas Instruments -> (none); Manufacturer_Part_Number TLA431AIDBZR -> (none); Mouser Part Number 595-TLA431AIDBZR -> (none); Mouser Price/Stock https://www.mouser.co.uk/ProductDetail/Texas-Instruments/TL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 -> (none)
- R52, R54: Distribuidor Mouser -> (none); Link https://pt.mouser.com/ProductDetail/Vishay/CRCW060320K0FKEC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 -> (none); MPN (none) -> CRCW060320K0FKEC; Ref CRCW060320K0FKEC -> (none)
- R53: Distribuidor Mouser -> (none); Link https://pt.mouser.com/ProductDetail/Bourns/CMP1206-FX-1001E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 -> (none); MPN (none) -> CMP1206-FX-1001ELF; Ref CMP1206-FX-1001ELF -> (none)
- R56: Distribuidor Mouser -> (none); Link https://pt.mouser.com/ProductDetail/Vishay/CRCW060354K9FKEA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 -> (none); MPN (none) -> CRCW060354K9FKEA; Ref CRCW060354K9FKEA -> (none)
- R57: Distribuidor Mouser -> (none); Link https://pt.mouser.com/ProductDetail/Panasonic/ERJ-PA3F7502V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 -> (none); MPN (none) -> ERJ-PA3F7502V; Ref ERJ-PA3F7502V -> (none)
- R59, R60, R61, R62, R63: Distribuidor Mouser -> (none); Link https://pt.mouser.com/ProductDetail/Vishay-Draloric/RCS0603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 -> (none); MPN (none) -> RCS060310K0FKEA; Ref RCS060310K0FKEA -> (none)
- R64: Distribuidor Mouser -> (none); Link https://pt.mouser.com/ProductDetail/Vishay/CRCW080547R0JNEA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 -> (none); MPN (none) -> CRCW080547R0JNEAC; Ref CRCW080547R0JNEAC -> (none)
- R65: Distribuidor Mouser -> (none); Link https://pt.mouser.com/ProductDetail/Vishay/CRCW060338K3FKEA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 -> (none); MPN (none) -> CRCW060338K3FKEA; Ref CRCW060338K3FKEA -> (none)
- U4, U5: Distribuidor Mouser -> (none); Link https://pt.mouser.com/ProductDetail/Texas-Instruments/TLV18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 -> (none); MPN (none) -> TLV1805DBVR; Ref TLV1805DBVR -> (none)
