File: PCB/Power_Phase.kicad_sch (KiCad schematic)
At the start: 26 parts, among them T9 ZMPT101B, U12 IVY-CT-PCB-01-10A, U7 ADE7953xCP, Y5 GC0350016

Commit message: Implementação do novo circuito do Wleding detector; correcao dos campos dos componentes
Parts:
- removed R107, R108: 24K, Resistor_SMD:R_0603_1608Metric, symbol Device:R
- added R155, R99: 24K, Resistor_SMD:R_1206_3216Metric, symbol Device:R
- C105, C109, C112, C116: Distribuidor Mouser -> (none); Link https://pt.mouser.com/ProductDetail/Samsung-Electro-Mechani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 -> (none); MPN (none) -> CL10B104MB8NNNC; Ref CL10B104MB8NNNC -> (none)
- C106, C107: Distribuidor Mouser -> (none); Link https://pt.mouser.com/ProductDetail/Walsin/0603B333J500CT?q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 -> (none); MPN (none) -> 0603B333J500CT; Ref 0603B333J500CT -> (none)
- C108, C111, C115, C83: Distribuidor Mouser -> (none); Link https://pt.mouser.com/ProductDetail/Murata-Electronics/GRM2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 -> (none); MPN (none) -> GRM21BZ7YA475ME15L; Ref GRM21BZ7YA475ME15L -> (none)
- C110: Distribuidor Mouser -> (none); Link https://pt.mouser.com/ProductDetail/TAIYO-YUDEN/GMK316AB710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 -> (none); MPN (none) -> GMK316AB7106KL-TR; Ref GMK316AB7106KL-TR -> (none)
- C113, C114: Distribuidor Mouser -> (none); Link https://pt.mouser.com/ProductDetail/SEI-Stackpole/CML0603C0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 -> (none); MPN (none) -> CML0603C0G300JT50V; Ref CML0603C0G300JT50V -> (none)
- R103: footprint Resistor_SMD:R_0603_1608Metric -> Resistor_SMD:R_1206_3216Metric; Distribuidor Mouser -> (none); Link https://pt.mouser.com/ProductDetail/Panasonic/ERJ-PA3F2402V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 -> (none); MPN (none) -> ESR18EZPF2402; Ref ERJ-PA3F2402V -> (none)
- R104: footprint Resistor_SMD:R_0603_1608Metric -> Resistor_SMD:R_1206_3216Metric; MPN (none) -> ESR18EZPF2402
- R149: Destribuidor Mouser -> (none); Link https://pt.mouser.com/ProductDetail/Vishay/CRCW060336R0FKEA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 -> (none); MPN (none) -> CRCW060336R0FKEA; Ref CRCW060336R0FKEA -> (none)
- R150, R151: Distribuidor Mouser -> (none); Link https://pt.mouser.com/ProductDetail/Vishay/CRCW0603100RJNEA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 -> (none); MPN (none) -> CRCW0603100RJNEA; Ref CRCW0603100RJNEA -> (none)
- R152, R153: Distribuidor Mouser -> (none); Link https://pt.mouser.com/ProductDetail/Vishay-Draloric/RCS0603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 -> (none); MPN (none) -> RCS060310K0FKEA; Ref RCS060310K0FKEA -> (none)
- T9: Availability Not in stock -> (none); Check_prices https://www.snapeda.com/parts/ZMPT101B/Qingxian+Zeming+Lang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 -> (none); Description_1 Current-type Voltage Transformer -> (none); MANUFACTURER Qingxian Zeming Langxi Electronic -> (none); MAXIMUM_PACKAGE_HEIGHT 18.8mm -> (none); MF Qingxian Zeming Langxi Electronic -> (none); MP ZMPT101B -> (none); PARTREV NA -> (none); Price None -> (none); STANDARD Manufacturer Recommendations -> (none); SnapEDA_Link https://www.snapeda.com/parts/ZMPT101B/Qingxian+Zeming+Lang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 -> (none)
- U7: Distribuidor Mouser -> (none); Link https://pt.mouser.com/ProductDetail/Analog-Devices/ADE7953A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 -> (none); MPN (none) -> ADE7953ACPZ; Ref ADE7953ACPZ -> (none)
- Y5: Distribuidor Mouser -> (none); Link https://pt.mouser.com/ProductDetail/Diodes-Incorporated/GC0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 -> (none); MPN (none) -> GC0350016; Ref GC0350016 -> (none)
Connections:
- net at R104.1: now also R155.2
- net at R104.2: now also R99.1; no longer R103.1
- net at T9.1: now also R155.1
- new net: R103.1, R99.2
Other:
- moved on the sheet: T9

Commit message: Routing terminado; A corrigir violações; falta colocar as proteçãoes de inversão de polaridade; fusivél; TVS
Parts:
- added C85, C94: 33nF, Capacitor_SMD:C_0603_1608Metric_Pad1.08x0.95mm_HandSolder, symbol Device:C
- added R163: 4R99, Resistor_SMD:R_0603_1608Metric, symbol Device:R
- added R166, R169, R175, R178: 1K, Resistor_SMD:R_0603_1608Metric, symbol Device:R
- added R181: 49R9, Resistor_SMD:R_0603_1608Metric, symbol Device:R
- C110: value 10uF -> 1uF; MPN GMK316AB7106KL-TR -> CL10B105KB8NQNC
- R149: value 15R8 -> 4R99; MPN CRCW060336R0FKEA -> CRCW06034K99FKEAC
- R150: value 100R -> 49R9
Connections:
- net GND: now also C106.2, R149.1, R150.2, C85.1, C94.2, R163.2, R181.1; no longer C106.1
- net at R150.1, T9.4: now also R175.1; no longer C106.2, U7.12 (VP)
- net at R149.2, U12.1: now also R166.2; no longer U7.6 (IAN)
- new net: C85.2, R166.1, U7.6 (IAN)
- new net: C106.1, R175.2, U7.11 (VN)
- new net: C94.1, R169.1, U7.5 (IAP)
- new net: C107.2, R178.2, U7.12 (VP)
- new net: R163.1, R169.2, U12.2
- new net: R178.1, R181.2, T9.3
Other:
- note removed: "11kW 3PHASE -> 36R for current transformer R ->CRCW060336R0FKEA"
- moved on the sheet: C106, C107, R149, R150
