File: PCB/MCU.kicad_sch (KiCad schematic)
At the start: 12 parts, among them IC9 STM32C031C6T6, J2 Conn_01x05_Socket, SW1 SW_SPST, Y3 CX2016FB48000C0FZZH1

Commit message: Implementação do novo circuito do Wleding detector; correcao dos campos dos componentes
Parts:
- C41, C42: Distribuidor Mouser -> (none); Link https://pt.mouser.com/ProductDetail/YAGEO/CC0603BRNPO9BN4R0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 -> (none); MPN (none) -> CC0603BRNPO9BN4R0; Ref CC0603BRNPO9BN4R0 -> (none)
- C43, C44, C45: Distribuidor Mouser -> (none); Link https://pt.mouser.com/ProductDetail/Samsung-Electro-Mechani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 -> (none); MPN (none) -> CL10B104MB8NNNC; Ref CL10B104MB8NNNC -> (none)
- C46: Distribuidor Mouser -> (none); Link https://pt.mouser.com/ProductDetail/Walsin/0603B333J500CT?q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 -> (none); MPN (none) -> 0603B333J500CT; Ref 0603B333J500CT -> (none)
- IC9: Distribuidor Mouser -> (none); Link https://pt.mouser.com/ProductDetail/STMicroelectronics/STM3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 -> (none); MPN (none) -> STM32C031C6T6; Ref STM32C031C6T6 -> (none)
- R109: Distribuidor Mouser -> (none); Link https://pt.mouser.com/ProductDetail/YAGEO/RE0603FRE07150RL?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 -> (none); MPN (none) -> RE0603FRE07150RL; Ref RE0603FRE07150RL -> (none)
- SW1: Distribuidor Mouser -> (none); Link https://pt.mouser.com/ProductDetail/Omron-Electronics/B3U-1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 -> (none); MPN (none) -> B3U-1000PM; Ref B3U-1000PM -> (none)
- Y3: Distribuidor Mouser -> (none); Link https://pt.mouser.com/ProductDetail/KYOCERA-AVX/CX2016FB480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 -> (none); MPN (none) -> CX2016FB48000C0FZZH1; Ref CX2016FB48000C0FZZH1 -> (none)
Connections:
- net EN_WEL_DETEC: now reaches IC9.48 (PB9)
- no-connect marks 7 -> 6

Commit message: Routing terminado; A corrigir violações; falta colocar as proteçãoes de inversão de polaridade; fusivél; TVS
Connections:
- net RCD_TEST: now reaches IC9.47 (PB8)
- no-connect marks 6 -> 5
Changed lines of the file:
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@@
-	)
-	(no_connect
-		(at 151.13 81.28)
 	)
 	(no_connect
@@
 	(wire
 		(pts
+			(xy 139.7 73.66) (xy 151.13 73.66)
+		)
+		(stroke
+			(width 0)
+			(type default)
+		)
+	)
+	(wire
+		(pts
 			(xy 166.37 167.64) (xy 166.37 139.7)
 		)
@@
 		(pts
 			(xy 186.69 121.92) (xy 194.31 121.92)
+		)
+		(stroke
+			(width 0)
+			(type default)
+		)
+	)
+	(wire
+		(pts
+			(xy 151.13 73.66) (xy 151.13 81.28)
 		)
 		(stroke
@@
 		)
 	)
+	(hierarchical_label "RCD_TEST"
+		(shape input)
+		(at 139.7 73.66 180)
+		(effects
+			(font
+				(size 1.27 1.27)
+			)
+			(justify right)
+		)
+	)

Commit message: Layout finalizado
Connections:
- net RCD_TEST_DRIVE: now reaches IC9.46 (PB7)
- no-connect marks 5 -> 4
Changed lines of the file:
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@@
 		(at 156.21 81.28)
 	)
-	(no_connect
-		(at 153.67 81.28)
-	)
 	(wire
 		(pts
@@
 	(wire
 		(pts
+			(xy 153.67 71.12) (xy 153.67 81.28)
+		)
+		(stroke
+			(width 0)
+			(type default)
+		)
+	)
+	(wire
+		(pts
 			(xy 186.69 109.22) (xy 201.93 109.22)
 		)
@@
 		(pts
 			(xy 85.09 77.47) (xy 99.06 77.47)
+		)
+		(stroke
+			(width 0)
+			(type default)
+		)
+	)
+	(wire
+		(pts
+			(xy 139.7 71.12) (xy 153.67 71.12)
 		)
 		(stroke
@@
 		)
 	)
+	(hierarchical_label "RCD_TEST_DRIVE"
+		(shape input)
+		(at 139.7 71.12 180)
+		(effects
+			(font
+				(size 1.27 1.27)
+			)
+			(justify right)
+		)
+	)
