File: PCB/Welding_Contact_Detector.kicad_sch (KiCad schematic)
At the start: 26 parts, among them IC33 LM4040C30FTA, IC34 NCS2200SN1T1G, IC35 VO618A-3X017T, IC36 74LVC1G17GW,125

Commit message: Implementação do novo circuito do Wleding detector; correcao dos campos dos componentes
Parts:
- removed C136: 100nF, Capacitor_THT:C_Rect_L18.0mm_W5.0mm_P15.00mm_FKS3_FKP3, symbol Device:C
- removed C137: 100uF, Capacitor_SMD:C_Elec_8x10.2, symbol Device:C_Polarized
- removed C138: 220nF, Capacitor_SMD:C_0603_1608Metric, symbol Device:C
- removed C139: 330pF, Capacitor_SMD:C_0603_1608Metric, symbol Device:C
- removed C140: 1uF, Capacitor_SMD:C_0603_1608Metric_Pad1.08x0.95mm_HandSolder, symbol Device:C
- removed C141: 0.1uF, Capacitor_SMD:C_0603_1608Metric, symbol Device:C
- removed D35: 5.1V, Diode_SMD:D_SOD-123, symbol Device:D_Schottky_Dual_CommonAnode_AKK_Split
- removed D36: RS1MFP, Diode_SMD:D_SOD-123, symbol Device:D
- removed D37: BAT54S, Package_TO_SOT_SMD:SOT-23, symbol Diode:BAT54S
- removed IC33: LM4040C30FTA, Package_TO_SOT_SMD:SOT-23-3, symbol LM4040C30FTA:LM4040C30FTA
- removed IC34: NCS2200SN1T1G, FOOTPRINTS:SOT95P275X110-5N, symbol NCS2200SN1T1G:NCS2200SN1T1G
- removed IC35: VO618A-3X017T, FOOTPRINTS:SMD-4_OPTION_7, symbol VO618A-3X017T:VO618A-3X017T
- removed IC36: 74LVC1G17GW,125, FOOTPRINTS:SOT95P285X140-5N, symbol 74LVC1G17GW_125:74LVC1G17GW,125
- removed R176, R177, R188: 1K, Resistor_SMD:R_1206_3216Metric, symbol Device:R
- removed R178, R185: 470K, Resistor_SMD:R_1206_3216Metric, symbol Device:R
- removed R179: 750R, Resistor_SMD:R_0603_1608Metric, symbol Device:R
- removed R180, R181: 10M, Resistor_SMD:R_0805_2012Metric_Pad1.20x1.40mm_HandSolder, symbol Device:R
- removed R182: 200K, Resistor_SMD:R_0603_1608Metric, symbol Device:R
- removed R183, R184: 47K, Resistor_SMD:R_0603_1608Metric, symbol Device:R
- removed R186: 1.8K, Resistor_SMD:R_0603_1608Metric, symbol Device:R
- removed R187: 100k, Resistor_SMD:R_0603_1608Metric, symbol Device:R
- added C23: 100nF, Capacitor_THT:C_Rect_L18.0mm_W5.0mm_P15.00mm_FKS3_FKP3, symbol Device:C
- added C24: 220uF, Capacitor_THT:CP_Radial_D8.0mm_P3.50mm, symbol Device:C_Polarized
- added C25: 220nF, Capacitor_SMD:C_0603_1608Metric, symbol Device:C
- added C27: 470pF, Capacitor_SMD:C_0603_1608Metric, symbol Device:C
- added C28: 47nF, Capacitor_SMD:C_0603_1608Metric, symbol Device:C
- added C29: 1uF, Capacitor_SMD:C_0603_1608Metric, symbol Device:C
- added C30: 100nF, Capacitor_SMD:C_0603_1608Metric, symbol Device:C
- added D16, D25: RS1MFP, Diode_SMD:D_SOD-123, symbol Device:D
- added D28: SMAJ400A, FOOTPRINTS:DIOM5026X229N, symbol SMAJ400A:SMAJ400A
- added D7: 5V6, Diode_SMD:D_SOD-123, symbol Device:D_Schottky_Dual_CommonAnode_AKK_Split
- added IC15, IC18: VO618A-3X017T, FOOTPRINTS:SMD-4_OPTION_7, symbol VO618A-3X017T:VO618A-3X017T
- added IC16: LM4040C30FTA, Package_TO_SOT_SMD:SOT-23-3, symbol LM4040C30FTA:LM4040C30FTA
- added IC17: MCP6541RT-I_OT, FOOTPRINTS:SOT95P280X145-5N, symbol MCP6541RT-I_OT:MCP6541RT-I_OT
- added IC20: 74LVC1G17GW,125, FOOTPRINTS:SOT65P212X110-5N, symbol 74LVC1G17GW_125:74LVC1G17GW,125
- added Q7: DMN60H080DS, Package_TO_SOT_SMD:SOT-23-3, symbol BSS127IXTSA1:BSS127IXTSA1
- added R45, R46: 1k, Resistor_SMD:R_1206_3216Metric, symbol Device:R
- added R47: 470k, Resistor_SMD:R_1206_3216Metric, symbol Device:R
- added R48: 2K2, Resistor_SMD:R_0603_1608Metric, symbol Device:R
- added R49: 1K5, Resistor_SMD:R_0603_1608Metric, symbol Device:R
- added R50: 10K, Resistor_SMD:R_0603_1608Metric, symbol Device:R
- added R66: 39R, Resistor_SMD:R_0603_1608Metric, symbol Device:R
- added R68, R69: 22K, Resistor_THT:R_Axial_DIN0411_L9.9mm_D3.6mm_P12.70mm_Horizontal, symbol Device:R
- added R70: 68K, Resistor_SMD:R_0603_1608Metric, symbol Device:R
- added R71: 8K87, Resistor_SMD:R_0603_1608Metric, symbol Device:R
- added R72: 470k, Resistor_SMD:R_0603_1608Metric, symbol Device:R
- added R73: 1K8, Resistor_SMD:R_0603_1608Metric, symbol Device:R
- added R74: 100K, Resistor_SMD:R_0603_1608Metric, symbol Device:R
- added R75: 4K7, Resistor_SMD:R_0603_1608Metric, symbol Device:R
- added TP12, TP13, TP14, TP6, TP7: TestPoint, Connector_PinHeader_2.54mm:PinHeader_1x01_P2.54mm_Vertical, symbol Connector:TestPoint
Connections:
- net +3V3: now also C30.1, IC18.4 (C_2), IC20.5 (VCC)
- net GND: now also C29.2, C30.2, IC15.2 (C_1), IC20.3 (GND), R74.1
- net Line_RelayIN: now also R45.2
- net Neutral_RelayIN: now also C24.2, C25.2, C27.2, C28.2, D28.2 (A), D7.1 (A), IC16.2 (A_1), IC17.5 (VSS), R50.2, R66.2, R71.2, TP7.1
- net SW_CLOSED_STATE: now also IC20.4 (Y)
- net Sw_Line: now also R68.1, R69.1
- new net: C23.1, D16.2 (A), D7.2 (K), R47.1
- new net: D25.1 (K), D28.1 (K), Q7.3 (D)
- new net: D25.2 (A), R68.2, R69.2
- new net: IC15.1 (A), R48.1
- new net: C27.1, IC15.3 (E), Q7.1 (G), R50.1
- new net: C29.1, IC20.2 (A), R75.1
- new net: R45.1, R46.2
- new net: C28.1, IC17.4 (VIN-), Q7.2 (S), R66.1, TP6.1
- new net: IC18.3 (E), R74.2, R75.2
- new net: IC18.1 (A), R73.2
- new net: IC17.1 (OUT), IC18.2 (C_1), R72.1, TP12.1
- new net: IC17.3 (VIN+), R70.2, R71.1, R72.2
- new net: C23.2, R46.1, R47.2
- new net +3V_n: C25.1, IC16.1 (K), IC17.2 (VDD), R49.1, R70.1, R73.1, TP14.1
- new net +5V_n: C24.1, D16.1 (K), IC15.4 (C_2), R49.2, TP13.1
- new net ENABLE: R48.2
Other:
- note removed: "CL10B105KB8NQNC"

Commit message: Layout finalizado
Parts:
- removed R69: 22K, Resistor_THT:R_Axial_DIN0411_L9.9mm_D3.6mm_P12.70mm_Horizontal, symbol Device:R
- removed TP12, TP13, TP14, TP6, TP7: TestPoint, Connector_PinHeader_2.54mm:PinHeader_1x01_P2.54mm_Vertical, symbol Connector:TestPoint
