File: PCB/Charger_Power_BOARD_V_0_7_0.kicad_pcb (KiCad board)
At the start: 4 copper layers, 205 x 105.5 mm, 366 parts, among them IC10 TLA431AIDBZR, IC15 VO618A-3X017T, IC16 LM4040C30FTA, IC17 MCP6541RT-I_OT, IC18 VO618A-3X017T, IC19 TPS54302DDCT, IC20 74LVC1G17GW,125, IC21 VO618A-3X017T, IC22 LM4040C30FTA, IC23 MCP6541RT-I_OT, IC24 VO618A-3X017T, IC25 74LVC1G17GW,125, IC26 VO618A-3X017T, IC27 LM4040C30FTA, IC28 LM75BD,118, IC45 MCP6541RT-I_OT, IC46 VO618A-3X017T, IC47 74LVC1G17GW,125, IC48 VO618A-3X017T, IC49 LM4040C30FTA, IC50 MCP6541RT-I_OT, IC51 VO618A-3X017T, IC52 74LVC1G17GW,125, IC9 STM32C031C6T6, J1 AMT0440005TH0000G, J10 AMT0440005TH0000G, J11 AMT0440005TH0000G, J12 AMT0440005TH0000G, J13 AMT0440005TH0000G, J14 AMT0440005TH0000G, J15 AMT0440005TH0000G, J18 Conn_01x03_Pin, J19 Screw_Terminal_01x02, J2 Conn_01x05_Socket, J20 Screw_Terminal_01x02, J3 AMT0440005TH0000G, J4 Conn_01x04_Socket, J5 AMT0440005TH0000G, J6 B6B-XH-A_LF__SN_, J7 AMT0440005TH0000G, J8 Conn_01x02_Socket, J9 B6B-XH-A_LF__SN_, K5 Relay_IM_NE801A, K6 Relay_IM_NE801A, Q1 BSS84, Q10 DMN60H080DS, Q11 BSS316N H6327, Q2 SQD50P04-13L_T4GE3, Q5 BSS316N H6327, Q6 BSS316N H6327, Q7 DMN60H080DS, Q8 DMN60H080DS, Q9 DMN60H080DS, SW1 SW_SPST, T11 ZMPT101B, T7 ZMPT101B, T9 ZMPT101B, U1 THVD1400DR, U10 IVY-CT-PCB-01-10A, U11 DRV8220DRL, U12 IVY-CT-PCB-01-10A, U13 IVY-CT-PCB-01-10A, U4 TLV1805DBVR, U5 TLV1805DBVR, U6 ADE7953xCP, U7 ADE7953xCP, U8 RCD MD0630STA-P, U9 ADE7953xCP, Y3 CX2016FB48000C0FZZH1, Y4 GC0350016, Y5 GC0350016, Y6 GC0350016

Commit message: panelização feita, falta trocar o user_commnts para edge cuts
Other:
- outline, holes or cut-outs redrawn
