File: PCB_PANELIZE/Charger_Power_BOARD_V_0_7_0_panelize.kicad_pcb (KiCad board)
At the start: 4 copper layers, 205 x 105.5 mm, 366 parts, among them IC10 TLA431AIDBZR, IC15 VO618A-3X017T, IC16 LM4040C30FTA, IC17 MCP6541RT-I_OT, IC18 VO618A-3X017T, IC19 TPS54302DDCT, IC20 74LVC1G17GW,125, IC21 VO618A-3X017T, IC22 LM4040C30FTA, IC23 MCP6541RT-I_OT, IC24 VO618A-3X017T, IC25 74LVC1G17GW,125, IC26 VO618A-3X017T, IC27 LM4040C30FTA, IC28 LM75BD,118, IC45 MCP6541RT-I_OT, IC46 VO618A-3X017T, IC47 74LVC1G17GW,125, IC48 VO618A-3X017T, IC49 LM4040C30FTA, IC50 MCP6541RT-I_OT, IC51 VO618A-3X017T, IC52 74LVC1G17GW,125, IC9 STM32C031C6T6, J1 AMT0440005TH0000G, J10 AMT0440005TH0000G, J11 AMT0440005TH0000G, J12 AMT0440005TH0000G, J13 AMT0440005TH0000G, J14 AMT0440005TH0000G, J15 AMT0440005TH0000G, J18 Conn_01x03_Pin, J19 Screw_Terminal_01x02, J2 Conn_01x05_Socket, J20 Screw_Terminal_01x02, J3 AMT0440005TH0000G, J4 Conn_01x04_Socket, J5 AMT0440005TH0000G, J6 B6B-XH-A_LF__SN_, J7 AMT0440005TH0000G, J8 Conn_01x02_Socket, J9 B6B-XH-A_LF__SN_, K5 Relay_IM_NE801A, K6 Relay_IM_NE801A, Q1 BSS84, Q10 DMN60H080DS, Q11 BSS316N H6327, Q2 SQD50P04-13L_T4GE3, Q5 BSS316N H6327, Q6 BSS316N H6327, Q7 DMN60H080DS, Q8 DMN60H080DS, Q9 DMN60H080DS, SW1 SW_SPST, T11 ZMPT101B, T7 ZMPT101B, T9 ZMPT101B, U1 THVD1400DR, U10 IVY-CT-PCB-01-10A, U11 DRV8220DRL, U12 IVY-CT-PCB-01-10A, U13 IVY-CT-PCB-01-10A, U4 TLV1805DBVR, U5 TLV1805DBVR, U6 ADE7953xCP, U7 ADE7953xCP, U8 RCD MD0630STA-P, U9 ADE7953xCP, Y3 CX2016FB48000C0FZZH1, Y4 GC0350016, Y5 GC0350016, Y6 GC0350016

Commit message: panelização feita, falta trocar o user_commnts para edge cuts
Parts:
- removed the C1 at (204.1, 14.0)
- removed the C100 at (263.3, 67.7)
- removed the C103 at (238.5, 22.0)
- removed the C104 at (131.7, 16.2)
- removed the C105 at (116.3, 55.1)
- removed the C106 at (116.4, 61.7)
- removed the C107 at (118.8, 59.3)
- removed the C108 at (102.0, 57.2)
- removed the C109 at (104.7, 58.6)
- removed the C110 at (102.6, 55.0)
- removed the C111 at (115.1, 52.7)
- removed the C112 at (113.7, 53.8)
- removed the C113 at (112.4, 51.0)
- removed the C114 at (111.3, 49.9)
- removed the C115 at (115.4, 57.9)
- removed the C116 at (113.0, 56.7)
- removed the C117 at (92.6, 56.2)
- removed the C118 at (91.5, 54.8)
- removed the C119 at (91.7, 61.7)
- removed the C120 at (94.1, 59.3)
- removed the C121 at (77.0, 57.2)
- removed the C122 at (79.5, 58.7)
- removed the C123 at (77.6, 55.0)
- removed the C124 at (90.1, 52.6)
- removed the C125 at (88.7, 53.7)
- removed the C126 at (87.5, 51.1)
- removed the C127 at (86.4, 50.0)
- removed the C128 at (90.3, 57.8)
- removed the C129 at (88.0, 56.5)
- removed the C2 at (204.9, 16.0)
- removed the C23 at (199.5, 51.0)
- removed the C24 at (213.1, 36.8)
- removed the C25 at (190.2, 34.5)
- removed the C26 at (179.3, 51.4)
- removed the C27 at (200.4, 31.7)
- removed the C28 at (196.3, 29.6)
- removed the C29 at (176.9, 25.3)
- removed the C30 at (172.3, 26.1)
- removed the C31 at (185.2, 55.1)
- removed the C32 at (188.8, 63.9)
- removed the C33 at (188.0, 47.0)
- removed the C34 at (194.5, 38.5)
- removed the C35 at (173.3, 35.4)
- removed the C36 at (170.0, 27.7)
- removed the C37 at (237.5, 51.5)
- removed the C38 at (233.0, 43.7)
- removed the C39 at (228.5, 46.5)
- removed the C40 at (224.0, 43.0)
- removed the C41 at (118.8, 22.0)
- removed the C42 at (115.5, 21.9)
- removed the C43 at (115.1, 26.3)
- removed the C44 at (114.0, 27.4)
- removed the C45 at (112.9, 28.5)
- removed the C46 at (110.4, 29.2)
- removed the C47 at (173.1, 18.5)
- removed the C48 at (170.5, 17.0)
- removed the C49 at (178.4, 22.9)
- removed the C50 at (144.4, 26.8)
- removed the C51 at (135.2, 19.5)
- removed the C52 at (135.2, 21.0)
- removed the C53 at (146.4, 34.6)
- removed the C54 at (146.8, 20.3)
- removed the C55 at (143.4, 20.4)
- removed the C56 at (129.0, 23.5)
- removed the C57 at (140.6, 26.8)
- removed the C58 at (235.8, 35.3)
- removed the C59 at (213.5, 27.4)
- removed the C60 at (210.5, 28.8)
- removed the C61 at (256.0, 48.0)
- removed the C62 at (250.7, 48.0)
- removed the C63 at (247.5, 42.0)
- removed the C64 at (254.9, 30.5)
- removed the C65 at (255.5, 40.0)
- removed the C66 at (239.4, 29.7)
- removed the C67 at (234.2, 26.8)
- removed the C70 at (127.6, 55.0)
- removed the C71 at (140.4, 57.9)
- removed the C72 at (138.1, 56.5)
- removed the C73 at (140.8, 61.7)
- removed the C74 at (143.2, 59.3)
- removed the C75 at (137.4, 50.9)
- removed the C76 at (136.3, 49.8)
- removed the C77 at (142.7, 56.3)
- removed the C78 at (141.3, 55.1)
- removed the C79 at (127.0, 57.3)
- removed the C80 at (129.7, 58.6)
- removed the C81 at (140.1, 52.6)
- removed the C82 at (138.7, 53.7)
- removed the C83 at (117.8, 56.3)
- removed the C84 at (235.2, 22.5)
- removed the C85 at (110.9, 59.5)
- removed the C86 at (95.3, 18.2)
- removed the C87 at (93.0, 18.2)
- removed the C88 at (101.2, 21.8)
- removed the C89 at (100.2, 29.6)
- removed the C90 at (93.0, 24.5)
- removed the C91 at (91.0, 23.9)
- removed the C92 at (85.9, 59.5)
- removed the C93 at (136.0, 59.4)
- removed the C94 at (104.5, 61.1)
- removed the C95 at (79.7, 61.1)
- removed the C96 at (129.5, 61.0)
- removed the C97 at (167.9, 78.0)
- removed the C98 at (165.9, 77.3)
- removed the C99 at (261.5, 64.4)
- removed the D1 at (213.1, 20.4)
- removed the D10 at (179.9, 18.9)
- removed the D11 at (146.0, 24.0)
- removed the D12 at (144.0, 34.5)
- removed the D13 at (142.5, 24.0)
- removed the D14 at (139.0, 24.0)
- removed the D16 at (205.5, 46.5)
- removed the D17 at (72.1, 58.7)
- removed the D18 at (171.5, 65.0)
- removed the D19 at (145.5, 14.0)
- removed the D2 at (100.1, 38.0)
- removed the D20 at (136.5, 14.0)
- removed the D22 at (271.0, 47.2)
- removed the D25 at (203.0, 38.6)
- removed the D28 at (203.4, 35.5)
- removed the D29 at (186.3, 60.9)
- removed the D3 at (101.5, 34.5)
- removed the D30 at (183.8, 60.9)
- removed the D31 at (190.7, 47.6)
- removed the D48 at (197.1, 36.7)
- removed the D49 at (238.5, 45.1)
- removed the D50 at (235.0, 47.5)
- removed the D51 at (221.5, 39.0)
- removed the D52 at (220.0, 44.0)
- removed the D53 at (248.0, 55.0)
- removed the D54 at (251.0, 55.0)
- removed the D55 at (263.2, 34.0)
- removed the D56 at (259.5, 42.0)
- removed the D7 at (214.2, 44.0)
- removed the F1 at (76.9, 35.2)
- removed the G*** at (74.9, 14.1)
- removed the H10 at (96.5, 93.0)
- removed the H11 at (214.5, 62.5)
- removed the H12 at (81.3, 94.0)
- removed the H13 at (202.0, 62.5)
- removed the H14 at (111.0, 93.0)
- removed the H15 at (226.5, 62.5)
- removed the H16 at (126.0, 93.0)
- removed the H17 at (240.0, 62.5)
- removed the H19 at (262.8, 98.9)
- removed the H5 at (142.0, 93.0)
- removed the H6 at (267.9, 23.8)
- removed the H7 at (267.9, 62.5)
- removed the H8 at (74.7, 23.8)
- removed the H9 at (74.7, 84.1)
- removed the IC10 at (144.0, 30.5)
- removed the IC15 at (180.0, 35.5)
- removed the IC16 at (193.2, 34.5)
- removed the IC17 at (193.2, 29.5)
- removed the IC18 at (180.0, 30.5)
- removed the IC19 at (98.2, 24.1)
- removed the IC20 at (173.2, 23.1)
- removed the IC21 at (180.0, 45.5)
- removed the IC22 at (191.8, 62.9)
- removed the IC23 at (191.5, 38.5)
- removed the IC24 at (180.0, 40.5)
- removed the IC25 at (170.7, 31.1)
- removed the IC26 at (222.0, 31.5)
- removed the IC27 at (225.5, 46.5)
- removed the IC28 at (126.3, 18.2)
- removed the IC45 at (232.8, 35.4)
- removed the IC46 at (222.0, 26.5)
- removed the IC47 at (210.7, 26.6)
- removed the IC48 at (247.5, 28.6)
- removed the IC49 at (250.5, 42.0)
- removed the IC50 at (255.5, 37.0)
- removed the IC51 at (247.5, 33.5)
- removed the IC52 at (236.5, 28.5)
- removed the IC9 at (120.6, 31.2)
- removed the J1 at (113.2, 111.2)
- removed the J10 at (145.2, 111.2)
- removed the J11 at (231.3, 111.2)
- removed the J12 at (215.3, 111.2)
- removed the J13 at (199.3, 111.2)
- removed the J14 at (247.3, 111.2)
- removed the J15 at (267.9, 105.8)
- removed the J18 at (255.5, 18.0)
- removed the J19 at (193.5, 18.3)
- removed the J2 at (134.6, 38.7)
- removed the J20 at (74.7, 41.5)
- removed the J3 at (97.2, 111.2)
- removed the J4 at (198.4, 24.1)
- removed the J5 at (81.2, 111.2)
- removed the J6 at (210.5, 16.0)
- removed the J7 at (129.2, 111.2)
- removed the J8 at (221.4, 20.5)
- removed the J9 at (228.5, 16.0)
- removed the K5 at (218.3, 69.0)
- removed the K6 at (223.7, 95.0)
- removed the L1 at (85.5, 21.2)
- removed the Q1 at (163.4, 15.9)
- removed the Q10 at (259.9, 30.5)
- removed the Q11 at (156.7, 15.9)
- removed the Q2 at (90.7, 36.1)
- removed the Q5 at (171.5, 59.4)
- removed the Q6 at (271.1, 41.1)
- removed the Q7 at (202.9, 31.2)
- removed the Q8 at (188.0, 44.0)
- removed the Q9 at (226.5, 40.5)
- removed the R1 at (200.8, 15.9)
- removed the R100 at (85.0, 81.0)
- removed the R101 at (120.0, 83.0)
- removed the R102 at (146.5, 62.5)
- removed the R103 at (100.0, 86.0)
- removed the R104 at (108.7, 83.0)
- removed the R105 at (146.5, 47.0)
- removed the R106 at (217.5, 21.5)
- removed the R107 at (90.0, 81.0)
- removed the R108 at (123.8, 83.0)
- removed the R109 at (72.1, 55.6)
- removed the R110 at (171.6, 56.5)
- removed the R111 at (104.0, 24.1)
- removed the R112 at (271.1, 38.1)
- removed the R113 at (100.3, 26.6)
- removed the R114 at (146.5, 45.5)
- removed the R115 at (214.2, 30.9)
- removed the R116 at (231.0, 48.0)
- removed the R117 at (222.5, 43.0)
- removed the R118 at (226.5, 43.5)
- removed the R119 at (242.0, 53.4)
- removed the R120 at (151.8, 16.7)
- removed the R121 at (229.5, 35.0)
- removed the R122 at (227.9, 36.9)
- removed the R123 at (232.2, 32.8)
- removed the R124 at (229.5, 32.0)
- removed the R125 at (215.2, 27.4)
- removed the R126 at (214.5, 25.0)
- removed the R127 at (249.5, 67.0)
- removed the R128 at (254.5, 67.0)
- removed the R129 at (251.0, 60.0)
- removed the R130 at (239.7, 27.3)
- removed the R131 at (253.5, 42.5)
- removed the R132 at (256.9, 30.5)
- removed the R133 at (258.4, 33.2)
- removed the R134 at (263.5, 50.9)
- removed the R136 at (255.5, 42.5)
- removed the R137 at (255.5, 45.0)
- removed the R138 at (255.2, 34.0)
- removed the R139 at (250.0, 39.5)
- removed the R140 at (240.9, 29.7)
- removed the R141 at (242.5, 23.5)
- removed the R142 at (240.0, 22.0)
- removed the R143 at (184.3, 16.2)
- removed the R144 at (121.0, 19.4)
- removed the R145 at (121.0, 16.3)
- removed the R146 at (121.0, 17.9)
- removed the R147 at (148.5, 14.0)
- removed the R148 at (139.5, 14.0)
- removed the R149 at (112.6, 62.7)
- removed the R150 at (122.1, 62.6)
- removed the R151 at (103.4, 51.4)
- removed the R152 at (103.4, 53.0)
- removed the R153 at (108.2, 49.5)
- removed the R154 at (85.0, 87.0)
- removed the R155 at (111.9, 80.1)
- removed the R156 at (93.6, 82.7)
- removed the R157 at (128.0, 81.3)
- removed the R158 at (87.9, 62.7)
- removed the R159 at (97.4, 62.6)
- removed the R160 at (78.4, 51.4)
- removed the R161 at (78.4, 53.0)
- removed the R162 at (83.2, 49.5)
- removed the R163 at (107.7, 62.7)
- removed the R164 at (83.1, 62.7)
- removed the R165 at (132.7, 62.6)
- removed the R166 at (110.8, 61.1)
- removed the R167 at (86.1, 61.1)
- removed the R168 at (135.8, 61.0)
- removed the R169 at (107.7, 61.1)
- removed the R170 at (83.0, 61.1)
- removed the R171 at (132.7, 61.0)
- removed the R172 at (99.3, 40.4)
- removed the R173 at (166.0, 15.9)
- removed the R175 at (122.1, 61.0)
- removed the R176 at (97.4, 61.0)
- removed the R177 at (146.5, 60.9)
- removed the R178 at (122.1, 59.4)
- removed the R179 at (97.4, 59.4)
- removed the R180 at (146.5, 59.3)
- removed the R181 at (122.1, 57.8)
- removed the R182 at (97.4, 57.8)
- removed the R183 at (146.5, 57.7)
- removed the R2 at (209.2, 21.1)
- removed the R215 at (240.1, 32.0)
- removed the R27 at (146.3, 54.5)
- removed the R28 at (154.1, 16.0)
- removed the R3 at (209.2, 19.6)
- removed the R45 at (215.8, 55.1)
- removed the R46 at (211.1, 55.1)
- removed the R47 at (200.0, 46.5)
- removed the R48 at (173.1, 31.5)
- removed the R49 at (187.8, 34.0)
- removed the R50 at (198.9, 31.7)
- removed the R51 at (104.0, 25.6)
- removed the R52 at (172.9, 13.4)
- removed the R53 at (180.4, 15.8)
- removed the R54 at (175.9, 13.4)
- removed the R55 at (181.6, 21.4)
- removed the R56 at (181.5, 22.9)
- removed the R57 at (178.6, 21.4)
- removed the R58 at (147.0, 28.0)
- removed the R59 at (133.6, 26.1)
- removed the R60 at (136.3, 23.6)
- removed the R61 at (140.4, 29.6)
- removed the R62 at (136.3, 26.6)
- removed the R63 at (129.0, 22.0)
- removed the R64 at (133.5, 28.0)
- removed the R65 at (140.4, 31.1)
- removed the R66 at (206.2, 32.4)
- removed the R67 at (100.3, 28.1)
- removed the R68 at (196.2, 42.5)
- removed the R69 at (160.9, 16.1)
- removed the R70 at (190.2, 29.6)
- removed the R71 at (191.2, 32.0)
- removed the R72 at (187.8, 29.0)
- removed the R73 at (187.8, 31.8)
- removed the R74 at (176.9, 26.9)
- removed the R75 at (174.5, 26.1)
- removed the R76 at (192.1, 67.3)
- removed the R77 at (187.3, 67.0)
- removed the R78 at (183.8, 65.8)
- removed the R79 at (173.9, 49.8)
- removed the R80 at (188.8, 60.9)
- removed the R81 at (188.0, 48.5)
- removed the R82 at (190.6, 43.5)
- removed the R83 at (194.0, 59.4)
- removed the R84 at (159.3, 16.1)
- removed the R85 at (188.5, 39.5)
- removed the R86 at (190.9, 41.1)
- removed the R87 at (187.0, 39.5)
- removed the R88 at (187.7, 36.9)
- removed the R89 at (170.1, 35.4)
- removed the R90 at (171.7, 35.4)
- removed the R91 at (230.5, 55.5)
- removed the R92 at (225.5, 55.5)
- removed the R93 at (219.5, 50.0)
- removed the R94 at (128.4, 53.0)
- removed the R95 at (128.4, 51.4)
- removed the R96 at (137.5, 62.6)
- removed the R97 at (133.2, 49.5)
- removed the R98 at (116.0, 86.0)
- removed the R99 at (104.0, 83.0)
- removed the SW1 at (111.3, 33.4)
- removed the T11 at (177.9, 106.6)
- removed the T7 at (159.2, 88.8)
- removed the T9 at (159.2, 107.8)
- removed the U1 at (203.0, 19.5)
- removed the U10 at (143.8, 76.0)
- removed the U11 at (232.5, 22.5)
- removed the U12 at (118.8, 76.0)
- removed the U13 at (93.8, 76.0)
- removed the U4 at (173.5, 15.9)
- removed the U5 at (133.0, 23.5)
- removed the U6 at (134.0, 55.0)
- removed the U7 at (109.0, 55.0)
- removed the U8 at (148.4, 18.7)
- removed the U9 at (84.0, 55.0)
- removed the Y3 at (117.2, 23.5)
- removed the Y4 at (141.0, 48.0)
- removed the Y5 at (116.0, 48.0)
- removed the Y6 at (91.0, 48.0)
- added C1: 10uF, Capacitor_SMD:C_1206_3216Metric, F.Cu at (181.1, 28.5)
- added C1: 10uF, Capacitor_SMD:C_1206_3216Metric, F.Cu at (181.1, 134.0)
- added C100: 0.1uF, Capacitor_SMD:C_0603_1608Metric, F.Cu at (240.3, 82.2)
- added C100: 0.1uF, Capacitor_SMD:C_0603_1608Metric, F.Cu at (240.3, 187.7)
- added C103: 33nF, Capacitor_SMD:C_0603_1608Metric, F.Cu at (215.5, 142.0)
- added C103: 33nF, Capacitor_SMD:C_0603_1608Metric, F.Cu at (215.5, 36.5)
- added C104: 0.1uF, Capacitor_SMD:C_0603_1608Metric, F.Cu at (108.7, 136.2)
- added C104: 0.1uF, Capacitor_SMD:C_0603_1608Metric, F.Cu at (108.7, 30.7)
- added C105: 0.1uF, Capacitor_SMD:C_0603_1608Metric, F.Cu at (93.3, 69.6)
- added C105: 0.1uF, Capacitor_SMD:C_0603_1608Metric, F.Cu at (93.3, 175.1)
- added C106: 33nF, Capacitor_SMD:C_0603_1608Metric_Pad1.08x0.95mm_HandSolder, F.Cu at (93.4, 181.7)
- added C106: 33nF, Capacitor_SMD:C_0603_1608Metric_Pad1.08x0.95mm_HandSolder, F.Cu at (93.4, 76.2)
- added C107: 33nF, Capacitor_SMD:C_0603_1608Metric_Pad1.08x0.95mm_HandSolder, F.Cu at (95.8, 179.3)
- added C107: 33nF, Capacitor_SMD:C_0603_1608Metric_Pad1.08x0.95mm_HandSolder, F.Cu at (95.8, 73.8)
- added C108: 4.7uF, Capacitor_SMD:C_0805_2012Metric, F.Cu at (79.0, 71.7)
- added C108: 4.7uF, Capacitor_SMD:C_0805_2012Metric, F.Cu at (79.0, 177.2)
- added C109: 0.1uF, Capacitor_SMD:C_0603_1608Metric, F.Cu at (81.7, 178.6)
- added C109: 0.1uF, Capacitor_SMD:C_0603_1608Metric, F.Cu at (81.7, 73.1)
- added C110: 1uF, Capacitor_SMD:C_1206_3216Metric, F.Cu at (79.6, 175.0)
- added C110: 1uF, Capacitor_SMD:C_1206_3216Metric, F.Cu at (79.6, 69.5)
- added C111: 4.7uF, Capacitor_SMD:C_0805_2012Metric, F.Cu at (92.1, 172.7)
- added C111: 4.7uF, Capacitor_SMD:C_0805_2012Metric, F.Cu at (92.1, 67.2)
- added C112: 0.1uF, Capacitor_SMD:C_0603_1608Metric, F.Cu at (90.7, 68.3)
- added C112: 0.1uF, Capacitor_SMD:C_0603_1608Metric, F.Cu at (90.7, 173.8)
- added C113: 30pF, Capacitor_SMD:C_0603_1608Metric_Pad1.08x0.95mm_HandSolder, F.Cu at (89.4, 171.0)
- added C113: 30pF, Capacitor_SMD:C_0603_1608Metric_Pad1.08x0.95mm_HandSolder, F.Cu at (89.4, 65.5)
- added C114: 30pF, Capacitor_SMD:C_0603_1608Metric_Pad1.08x0.95mm_HandSolder, F.Cu at (88.3, 169.9)
- added C114: 30pF, Capacitor_SMD:C_0603_1608Metric_Pad1.08x0.95mm_HandSolder, F.Cu at (88.3, 64.4)
- added C115: 4.7uF, Capacitor_SMD:C_0805_2012Metric, F.Cu at (92.4, 72.4)
- added C115: 4.7uF, Capacitor_SMD:C_0805_2012Metric, F.Cu at (92.4, 177.9)
- added C116: 0.1uF, Capacitor_SMD:C_0603_1608Metric, F.Cu at (90.0, 176.7)
- added C116: 0.1uF, Capacitor_SMD:C_0603_1608Metric, F.Cu at (90.0, 71.2)
- added C117: 4.7uF, Capacitor_SMD:C_0805_2012Metric, F.Cu at (69.6, 176.2)
- added C117: 4.7uF, Capacitor_SMD:C_0805_2012Metric, F.Cu at (69.6, 70.7)
- added C118: 0.1uF, Capacitor_SMD:C_0603_1608Metric, F.Cu at (68.5, 69.3)
- added C118: 0.1uF, Capacitor_SMD:C_0603_1608Metric, F.Cu at (68.5, 174.8)
- added C119: 33nF, Capacitor_SMD:C_0603_1608Metric_Pad1.08x0.95mm_HandSolder, F.Cu at (68.7, 76.2)
- added C119: 33nF, Capacitor_SMD:C_0603_1608Metric_Pad1.08x0.95mm_HandSolder, F.Cu at (68.7, 181.7)
- added C120: 33nF, Capacitor_SMD:C_0603_1608Metric_Pad1.08x0.95mm_HandSolder, F.Cu at (71.1, 73.8)
- added C120: 33nF, Capacitor_SMD:C_0603_1608Metric_Pad1.08x0.95mm_HandSolder, F.Cu at (71.1, 179.3)
- added C121: 4.7uF, Capacitor_SMD:C_0805_2012Metric, F.Cu at (54.0, 71.7)
- added C121: 4.7uF, Capacitor_SMD:C_0805_2012Metric, F.Cu at (54.0, 177.2)
- added C122: 0.1uF, Capacitor_SMD:C_0603_1608Metric, F.Cu at (56.5, 178.7)
- added C122: 0.1uF, Capacitor_SMD:C_0603_1608Metric, F.Cu at (56.5, 73.2)
- added C123: 1uF, Capacitor_SMD:C_1206_3216Metric, F.Cu at (54.6, 69.5)
- added C123: 1uF, Capacitor_SMD:C_1206_3216Metric, F.Cu at (54.6, 175.0)
- added C124: 4.7uF, Capacitor_SMD:C_0805_2012Metric, F.Cu at (67.1, 172.6)
- added C124: 4.7uF, Capacitor_SMD:C_0805_2012Metric, F.Cu at (67.1, 67.1)
- added C125: 0.1uF, Capacitor_SMD:C_0603_1608Metric, F.Cu at (65.7, 173.7)
- added C125: 0.1uF, Capacitor_SMD:C_0603_1608Metric, F.Cu at (65.7, 68.2)
- added C126: 30pF, Capacitor_SMD:C_0603_1608Metric_Pad1.08x0.95mm_HandSolder, F.Cu at (64.5, 171.1)
- added C126: 30pF, Capacitor_SMD:C_0603_1608Metric_Pad1.08x0.95mm_HandSolder, F.Cu at (64.5, 65.6)
- added C127: 30pF, Capacitor_SMD:C_0603_1608Metric_Pad1.08x0.95mm_HandSolder, F.Cu at (63.4, 64.5)
- added C127: 30pF, Capacitor_SMD:C_0603_1608Metric_Pad1.08x0.95mm_HandSolder, F.Cu at (63.4, 170.0)
- added C128: 4.7uF, Capacitor_SMD:C_0805_2012Metric, F.Cu at (67.3, 177.8)
- added C128: 4.7uF, Capacitor_SMD:C_0805_2012Metric, F.Cu at (67.3, 72.3)
- added C129: 0.1uF, Capacitor_SMD:C_0603_1608Metric, F.Cu at (65.0, 176.5)
- added C129: 0.1uF, Capacitor_SMD:C_0603_1608Metric, F.Cu at (65.0, 71.0)
- added C2: 0.1uF, Capacitor_SMD:C_0603_1608Metric, F.Cu at (181.9, 30.5)
- added C2: 0.1uF, Capacitor_SMD:C_0603_1608Metric, F.Cu at (181.9, 136.0)
- added C23: 100nF, Capacitor_THT:C_Rect_L18.0mm_W5.0mm_P15.00mm_FKS3_FKP3, F.Cu at (176.5, 171.0)
- added C23: 100nF, Capacitor_THT:C_Rect_L18.0mm_W5.0mm_P15.00mm_FKS3_FKP3, F.Cu at (176.5, 65.5)
- added C24: 220uF, Capacitor_THT:CP_Radial_D8.0mm_P3.50mm, F.Cu at (190.1, 156.8)
- added C24: 220uF, Capacitor_THT:CP_Radial_D8.0mm_P3.50mm, F.Cu at (190.1, 51.3)
- added C25: 220nF, Capacitor_SMD:C_0603_1608Metric, F.Cu at (167.2, 49.0)
- added C25: 220nF, Capacitor_SMD:C_0603_1608Metric, F.Cu at (167.2, 154.5)
- added C26: 100nF, Capacitor_THT:C_Rect_L18.0mm_W5.0mm_P15.00mm_FKS3_FKP3, F.Cu at (156.3, 65.8)
- added C26: 100nF, Capacitor_THT:C_Rect_L18.0mm_W5.0mm_P15.00mm_FKS3_FKP3, F.Cu at (156.3, 171.3)
- added C27: 470pF, Capacitor_SMD:C_0603_1608Metric, F.Cu at (177.4, 151.7)
- added C27: 470pF, Capacitor_SMD:C_0603_1608Metric, F.Cu at (177.4, 46.2)
- added C28: 47nF, Capacitor_SMD:C_0603_1608Metric, F.Cu at (173.3, 44.1)
- added C28: 47nF, Capacitor_SMD:C_0603_1608Metric, F.Cu at (173.3, 149.6)
- added C29: 1uF, Capacitor_SMD:C_0603_1608Metric, F.Cu at (153.9, 39.8)
- added C29: 1uF, Capacitor_SMD:C_0603_1608Metric, F.Cu at (153.9, 145.3)
- added C30: 100nF, Capacitor_SMD:C_0603_1608Metric, F.Cu at (149.3, 146.1)
- added C30: 100nF, Capacitor_SMD:C_0603_1608Metric, F.Cu at (149.3, 40.6)
- added C31: 220uF, Capacitor_THT:CP_Radial_D8.0mm_P3.50mm, F.Cu at (162.2, 175.1)
- added C31: 220uF, Capacitor_THT:CP_Radial_D8.0mm_P3.50mm, F.Cu at (162.2, 69.6)
- added C32: 220nF, Capacitor_SMD:C_0603_1608Metric, F.Cu at (165.8, 183.9)
- added C32: 220nF, Capacitor_SMD:C_0603_1608Metric, F.Cu at (165.8, 78.4)
- added C33: 470pF, Capacitor_SMD:C_0603_1608Metric, F.Cu at (165.0, 61.5)
- added C33: 470pF, Capacitor_SMD:C_0603_1608Metric, F.Cu at (165.0, 167.0)
- added C34: 47nF, Capacitor_SMD:C_0603_1608Metric, F.Cu at (171.5, 158.5)
- added C34: 47nF, Capacitor_SMD:C_0603_1608Metric, F.Cu at (171.5, 53.0)
- added C35: 1uF, Capacitor_SMD:C_0603_1608Metric, F.Cu at (150.3, 49.9)
- added C35: 1uF, Capacitor_SMD:C_0603_1608Metric, F.Cu at (150.3, 155.4)
- added C36: 100nF, Capacitor_SMD:C_0603_1608Metric, F.Cu at (147.0, 42.2)
- added C36: 100nF, Capacitor_SMD:C_0603_1608Metric, F.Cu at (147.0, 147.7)
- added C37: 100nF, Capacitor_THT:C_Rect_L18.0mm_W5.0mm_P15.00mm_FKS3_FKP3, F.Cu at (214.5, 66.0)
- added C37: 100nF, Capacitor_THT:C_Rect_L18.0mm_W5.0mm_P15.00mm_FKS3_FKP3, F.Cu at (214.5, 171.5)
- added C38: 220uF, Capacitor_THT:CP_Radial_D8.0mm_P3.50mm, F.Cu at (210.0, 163.7)
- added C38: 220uF, Capacitor_THT:CP_Radial_D8.0mm_P3.50mm, F.Cu at (210.0, 58.2)
- added C39: 220nF, Capacitor_SMD:C_0603_1608Metric, F.Cu at (205.5, 61.0)
- added C39: 220nF, Capacitor_SMD:C_0603_1608Metric, F.Cu at (205.5, 166.5)
- added C40: 470pF, Capacitor_SMD:C_0603_1608Metric, F.Cu at (201.0, 163.0)
- added C40: 470pF, Capacitor_SMD:C_0603_1608Metric, F.Cu at (201.0, 57.5)
- added C41: 4pF, Capacitor_SMD:C_0603_1608Metric_Pad1.08x0.95mm_HandSolder, F.Cu at (95.8, 36.5)
- added C41: 4pF, Capacitor_SMD:C_0603_1608Metric_Pad1.08x0.95mm_HandSolder, F.Cu at (95.8, 142.0)
- added C42: 4pF, Capacitor_SMD:C_0603_1608Metric_Pad1.08x0.95mm_HandSolder, F.Cu at (92.5, 36.4)
- added C42: 4pF, Capacitor_SMD:C_0603_1608Metric_Pad1.08x0.95mm_HandSolder, F.Cu at (92.5, 141.9)
- added C43: 0.1uF, Capacitor_SMD:C_0603_1608Metric, F.Cu at (92.1, 40.8)
- added C43: 0.1uF, Capacitor_SMD:C_0603_1608Metric, F.Cu at (92.1, 146.3)
- added C44: 0.1uF, Capacitor_SMD:C_0603_1608Metric, F.Cu at (91.0, 41.9)
- added C44: 0.1uF, Capacitor_SMD:C_0603_1608Metric, F.Cu at (91.0, 147.4)
- added C45: 0.1uF, Capacitor_SMD:C_0603_1608Metric, F.Cu at (89.9, 148.5)
- added C45: 0.1uF, Capacitor_SMD:C_0603_1608Metric, F.Cu at (89.9, 43.0)
- added C46: 33nF, Capacitor_SMD:C_0603_1608Metric_Pad1.08x0.95mm_HandSolder, F.Cu at (87.4, 149.2)
- added C46: 33nF, Capacitor_SMD:C_0603_1608Metric_Pad1.08x0.95mm_HandSolder, F.Cu at (87.4, 43.7)
- added C47: 0.1uF, Capacitor_SMD:C_0603_1608Metric, F.Cu at (150.1, 33.0)
- added C47: 0.1uF, Capacitor_SMD:C_0603_1608Metric, F.Cu at (150.1, 138.5)
- added C48: 0.1uF, Capacitor_SMD:C_0603_1608Metric, F.Cu at (147.5, 31.5)
- added C48: 0.1uF, Capacitor_SMD:C_0603_1608Metric, F.Cu at (147.5, 137.0)
- added C49: 220pF, Capacitor_SMD:C_0603_1608Metric_Pad1.08x0.95mm_HandSolder, F.Cu at (155.4, 37.5)
- added C49: 220pF, Capacitor_SMD:C_0603_1608Metric_Pad1.08x0.95mm_HandSolder, F.Cu at (155.4, 142.9)
- added C50: 1uF, Capacitor_SMD:C_0603_1608Metric_Pad1.08x0.95mm_HandSolder, F.Cu at (121.4, 146.8)
- added C50: 1uF, Capacitor_SMD:C_0603_1608Metric_Pad1.08x0.95mm_HandSolder, F.Cu at (121.4, 41.3)
- added C51: 1uF, Capacitor_SMD:C_0603_1608Metric_Pad1.08x0.95mm_HandSolder, F.Cu at (112.2, 139.5)
- added C51: 1uF, Capacitor_SMD:C_0603_1608Metric_Pad1.08x0.95mm_HandSolder, F.Cu at (112.2, 34.0)
- added C52: 10nF, Capacitor_SMD:C_0603_1608Metric_Pad1.08x0.95mm_HandSolder, F.Cu at (112.2, 35.5)
- added C52: 10nF, Capacitor_SMD:C_0603_1608Metric_Pad1.08x0.95mm_HandSolder, F.Cu at (112.2, 141.0)
- added C53: 1uF, Capacitor_SMD:C_0603_1608Metric_Pad1.08x0.95mm_HandSolder, F.Cu at (123.5, 154.6)
- added C53: 1uF, Capacitor_SMD:C_0603_1608Metric_Pad1.08x0.95mm_HandSolder, F.Cu at (123.5, 49.1)
- added C54: 1uF, Capacitor_SMD:C_0603_1608Metric_Pad1.08x0.95mm_HandSolder, F.Cu at (123.8, 140.3)
- added C54: 1uF, Capacitor_SMD:C_0603_1608Metric_Pad1.08x0.95mm_HandSolder, F.Cu at (123.8, 34.8)
- added C55: 1uF, Capacitor_SMD:C_0603_1608Metric_Pad1.08x0.95mm_HandSolder, F.Cu at (120.5, 34.9)
- added C55: 1uF, Capacitor_SMD:C_0603_1608Metric_Pad1.08x0.95mm_HandSolder, F.Cu at (120.5, 140.4)
- added C56: 1.5nF, Capacitor_SMD:C_0603_1608Metric_Pad1.08x0.95mm_HandSolder, F.Cu at (106.0, 143.5)
- added C56: 1.5nF, Capacitor_SMD:C_0603_1608Metric_Pad1.08x0.95mm_HandSolder, F.Cu at (106.0, 38.0)
- added C57: 1uF, Capacitor_SMD:C_0603_1608Metric_Pad1.08x0.95mm_HandSolder, F.Cu at (117.6, 41.3)
- added C57: 1uF, Capacitor_SMD:C_0603_1608Metric_Pad1.08x0.95mm_HandSolder, F.Cu at (117.6, 146.8)
- added C58: 47nF, Capacitor_SMD:C_0603_1608Metric, F.Cu at (212.8, 49.8)
- added C58: 47nF, Capacitor_SMD:C_0603_1608Metric, F.Cu at (212.8, 155.3)
- added C59: 1uF, Capacitor_SMD:C_0603_1608Metric, F.Cu at (190.5, 147.4)
- added C59: 1uF, Capacitor_SMD:C_0603_1608Metric, F.Cu at (190.5, 41.9)
- added C60: 100nF, Capacitor_SMD:C_0603_1608Metric, F.Cu at (187.5, 148.8)
- added C60: 100nF, Capacitor_SMD:C_0603_1608Metric, F.Cu at (187.5, 43.3)
- added C61: 100nF, Capacitor_THT:C_Rect_L18.0mm_W5.0mm_P15.00mm_FKS3_FKP3, F.Cu at (233.0, 168.0)
- added C61: 100nF, Capacitor_THT:C_Rect_L18.0mm_W5.0mm_P15.00mm_FKS3_FKP3, F.Cu at (233.0, 62.5)
- added C62: 220uF, Capacitor_THT:CP_Radial_D8.0mm_P3.50mm, F.Cu at (227.7, 62.5)
- added C62: 220uF, Capacitor_THT:CP_Radial_D8.0mm_P3.50mm, F.Cu at (227.7, 168.0)
- added C63: 220nF, Capacitor_SMD:C_0603_1608Metric, F.Cu at (224.5, 56.5)
- added C63: 220nF, Capacitor_SMD:C_0603_1608Metric, F.Cu at (224.5, 162.0)
- added C64: 470pF, Capacitor_SMD:C_0603_1608Metric, F.Cu at (231.9, 45.0)
- added C64: 470pF, Capacitor_SMD:C_0603_1608Metric, F.Cu at (231.9, 150.5)
- added C65: 47nF, Capacitor_SMD:C_0603_1608Metric, F.Cu at (232.5, 160.0)
- added C65: 47nF, Capacitor_SMD:C_0603_1608Metric, F.Cu at (232.5, 54.5)
- added C66: 1uF, Capacitor_SMD:C_0603_1608Metric, F.Cu at (216.4, 44.2)
- added C66: 1uF, Capacitor_SMD:C_0603_1608Metric, F.Cu at (216.4, 149.7)
- added C67: 100nF, Capacitor_SMD:C_0603_1608Metric, F.Cu at (211.2, 146.8)
- added C67: 100nF, Capacitor_SMD:C_0603_1608Metric, F.Cu at (211.2, 41.3)
- added C70: 1uF, Capacitor_SMD:C_1206_3216Metric, F.Cu at (104.6, 175.0)
- added C70: 1uF, Capacitor_SMD:C_1206_3216Metric, F.Cu at (104.6, 69.5)
- added C71: 4.7uF, Capacitor_SMD:C_0805_2012Metric, F.Cu at (117.4, 177.9)
- added C71: 4.7uF, Capacitor_SMD:C_0805_2012Metric, F.Cu at (117.4, 72.4)
- added C72: 0.1uF, Capacitor_SMD:C_0603_1608Metric, F.Cu at (115.1, 176.5)
- added C72: 0.1uF, Capacitor_SMD:C_0603_1608Metric, F.Cu at (115.1, 71.0)
- added C73: 33nF, Capacitor_SMD:C_0603_1608Metric_Pad1.08x0.95mm_HandSolder, F.Cu at (117.8, 76.2)
- added C73: 33nF, Capacitor_SMD:C_0603_1608Metric_Pad1.08x0.95mm_HandSolder, F.Cu at (117.8, 181.7)
- added C74: 33nF, Capacitor_SMD:C_0603_1608Metric_Pad1.08x0.95mm_HandSolder, F.Cu at (120.2, 179.3)
- added C74: 33nF, Capacitor_SMD:C_0603_1608Metric_Pad1.08x0.95mm_HandSolder, F.Cu at (120.2, 73.8)
- added C75: 30pF, Capacitor_SMD:C_0603_1608Metric_Pad1.08x0.95mm_HandSolder, F.Cu at (114.4, 170.9)
- added C75: 30pF, Capacitor_SMD:C_0603_1608Metric_Pad1.08x0.95mm_HandSolder, F.Cu at (114.4, 65.4)
- added C76: 30pF, Capacitor_SMD:C_0603_1608Metric_Pad1.08x0.95mm_HandSolder, F.Cu at (113.3, 169.8)
- added C76: 30pF, Capacitor_SMD:C_0603_1608Metric_Pad1.08x0.95mm_HandSolder, F.Cu at (113.3, 64.3)
- added C77: 4.7uF, Capacitor_SMD:C_0805_2012Metric, F.Cu at (119.7, 70.8)
- added C77: 4.7uF, Capacitor_SMD:C_0805_2012Metric, F.Cu at (119.7, 176.3)
- added C78: 0.1uF, Capacitor_SMD:C_0603_1608Metric, F.Cu at (118.3, 175.1)
- added C78: 0.1uF, Capacitor_SMD:C_0603_1608Metric, F.Cu at (118.3, 69.6)
- added C79: 4.7uF, Capacitor_SMD:C_0805_2012Metric, F.Cu at (104.0, 177.3)
- added C79: 4.7uF, Capacitor_SMD:C_0805_2012Metric, F.Cu at (104.0, 71.8)
- added C80: 0.1uF, Capacitor_SMD:C_0603_1608Metric, F.Cu at (106.7, 73.1)
- added C80: 0.1uF, Capacitor_SMD:C_0603_1608Metric, F.Cu at (106.7, 178.6)
- added C81: 4.7uF, Capacitor_SMD:C_0805_2012Metric, F.Cu at (117.1, 172.6)
- added C81: 4.7uF, Capacitor_SMD:C_0805_2012Metric, F.Cu at (117.1, 67.1)
- added C82: 0.1uF, Capacitor_SMD:C_0603_1608Metric, F.Cu at (115.7, 68.2)
- added C82: 0.1uF, Capacitor_SMD:C_0603_1608Metric, F.Cu at (115.7, 173.7)
- added C83: 4.7uF, Capacitor_SMD:C_0805_2012Metric, F.Cu at (94.8, 176.3)
- added C83: 4.7uF, Capacitor_SMD:C_0805_2012Metric, F.Cu at (94.8, 70.8)
- added C84: 0.1uF, Capacitor_SMD:C_0603_1608Metric, F.Cu at (212.2, 37.0)
- added C84: 0.1uF, Capacitor_SMD:C_0603_1608Metric, F.Cu at (212.2, 142.5)
- added C85: 33nF, Capacitor_SMD:C_0603_1608Metric_Pad1.08x0.95mm_HandSolder, F.Cu at (87.9, 179.5)
- added C85: 33nF, Capacitor_SMD:C_0603_1608Metric_Pad1.08x0.95mm_HandSolder, F.Cu at (87.9, 74.0)
- added C86: 22uF, Capacitor_SMD:C_1206_3216Metric, F.Cu at (72.3, 138.2)
- added C86: 22uF, Capacitor_SMD:C_1206_3216Metric, F.Cu at (72.3, 32.7)
- added C87: 22uF, Capacitor_SMD:C_1206_3216Metric, F.Cu at (70.0, 138.2)
- added C87: 22uF, Capacitor_SMD:C_1206_3216Metric, F.Cu at (70.0, 32.7)
- added C88: 0.1uF, Capacitor_SMD:C_0603_1608Metric, F.Cu at (78.2, 141.8)
- added C88: 0.1uF, Capacitor_SMD:C_0603_1608Metric, F.Cu at (78.2, 36.3)
- added C89: 44pF, Capacitor_SMD:C_0603_1608Metric, F.Cu at (77.2, 149.6)
- added C89: 44pF, Capacitor_SMD:C_0603_1608Metric, F.Cu at (77.2, 44.1)
- added C90: 10uF, Capacitor_SMD:C_1206_3216Metric, F.Cu at (70.0, 39.0)
- added C90: 10uF, Capacitor_SMD:C_1206_3216Metric, F.Cu at (70.0, 144.5)
- added C91: 0.1uF, Capacitor_SMD:C_0603_1608Metric, F.Cu at (68.0, 38.4)
- added C91: 0.1uF, Capacitor_SMD:C_0603_1608Metric, F.Cu at (68.0, 143.9)
- added C92: 33nF, Capacitor_SMD:C_0603_1608Metric_Pad1.08x0.95mm_HandSolder, F.Cu at (62.9, 179.5)
- added C92: 33nF, Capacitor_SMD:C_0603_1608Metric_Pad1.08x0.95mm_HandSolder, F.Cu at (62.9, 74.0)
- added C93: 33nF, Capacitor_SMD:C_0603_1608Metric_Pad1.08x0.95mm_HandSolder, F.Cu at (113.0, 73.9)
- added C93: 33nF, Capacitor_SMD:C_0603_1608Metric_Pad1.08x0.95mm_HandSolder, F.Cu at (113.0, 179.4)
- added C94: 33nF, Capacitor_SMD:C_0603_1608Metric_Pad1.08x0.95mm_HandSolder, F.Cu at (81.5, 75.6)
- added C94: 33nF, Capacitor_SMD:C_0603_1608Metric_Pad1.08x0.95mm_HandSolder, F.Cu at (81.5, 181.1)
- added C95: 33nF, Capacitor_SMD:C_0603_1608Metric_Pad1.08x0.95mm_HandSolder, F.Cu at (56.7, 181.1)
- added C95: 33nF, Capacitor_SMD:C_0603_1608Metric_Pad1.08x0.95mm_HandSolder, F.Cu at (56.7, 75.6)
- added C96: 33nF, Capacitor_SMD:C_0603_1608Metric_Pad1.08x0.95mm_HandSolder, F.Cu at (106.5, 75.5)
- added C96: 33nF, Capacitor_SMD:C_0603_1608Metric_Pad1.08x0.95mm_HandSolder, F.Cu at (106.5, 181.0)
- added C97: 0.1uF, Capacitor_SMD:C_0603_1608Metric, F.Cu at (144.9, 92.5)
- added C97: 0.1uF, Capacitor_SMD:C_0603_1608Metric, F.Cu at (144.9, 198.0)
- added C98: 10uF, Capacitor_SMD:C_1206_3216Metric, F.Cu at (142.9, 91.8)
- added C98: 10uF, Capacitor_SMD:C_1206_3216Metric, F.Cu at (142.9, 197.3)
- added C99: 10uF, Capacitor_SMD:C_1206_3216Metric, F.Cu at (238.5, 184.4)
- added C99: 10uF, Capacitor_SMD:C_1206_3216Metric, F.Cu at (238.5, 78.9)
- added D1: CDSOT23-SM712, Package_TO_SOT_SMD:SOT-23-3, F.Cu at (190.1, 34.9)
- added D1: CDSOT23-SM712, Package_TO_SOT_SMD:SOT-23-3, F.Cu at (190.1, 140.4)
- added D10: SMAJ14CA, Diode_SMD:D_SMA, F.Cu at (156.9, 33.4)
- added D10: SMAJ14CA, Diode_SMD:D_SMA, F.Cu at (156.9, 138.8)
- added D11: BAT54S, Package_TO_SOT_SMD:SOT-23, F.Cu at (123.0, 144.0)
- added D11: BAT54S, Package_TO_SOT_SMD:SOT-23, F.Cu at (123.0, 38.5)
- added D12: BAT54S, Package_TO_SOT_SMD:SOT-23, F.Cu at (121.0, 49.0)
- added D12: BAT54S, Package_TO_SOT_SMD:SOT-23, F.Cu at (121.0, 154.5)
- added D13: BAT54S, Package_TO_SOT_SMD:SOT-23, F.Cu at (119.5, 144.0)
- added D13: BAT54S, Package_TO_SOT_SMD:SOT-23, F.Cu at (119.5, 38.5)
- added D14: BAT54S, Package_TO_SOT_SMD:SOT-23, F.Cu at (116.0, 144.0)
- added D14: BAT54S, Package_TO_SOT_SMD:SOT-23, F.Cu at (116.0, 38.5)
- added D16: RS1MFP, Diode_SMD:D_SOD-123, F.Cu at (182.5, 61.0)
- added D16: RS1MFP, Diode_SMD:D_SOD-123, F.Cu at (182.5, 166.5)
- added D17: LED, LED_SMD:LED_0603_1608Metric, F.Cu at (49.1, 73.2)
- added D17: LED, LED_SMD:LED_0603_1608Metric, F.Cu at (49.1, 178.7)
- added D18: SS12, Diode_SMD:D_SMA, F.Cu at (148.5, 185.0)
- added D18: SS12, Diode_SMD:D_SMA, F.Cu at (148.5, 79.5)
- added D19: LED, LED_SMD:LED_0603_1608Metric, F.Cu at (122.5, 134.0)
- added D19: LED, LED_SMD:LED_0603_1608Metric, F.Cu at (122.5, 28.5)
- added D2: BZT52C13, Diode_SMD:D_SOD-123, F.Cu at (77.1, 158.0)
- added D2: BZT52C13, Diode_SMD:D_SOD-123, F.Cu at (77.1, 52.5)
- added D20: LED, LED_SMD:LED_0603_1608Metric, F.Cu at (113.5, 134.0)
- added D20: LED, LED_SMD:LED_0603_1608Metric, F.Cu at (113.5, 28.5)
- added D22: SS12, Diode_SMD:D_SMA, F.Cu at (248.0, 167.2)
- added D22: SS12, Diode_SMD:D_SMA, F.Cu at (248.0, 61.7)
- added D25: RS1MFP, Diode_SMD:D_SOD-123, F.Cu at (180.0, 158.6)
- added D25: RS1MFP, Diode_SMD:D_SOD-123, F.Cu at (180.0, 53.1)
- added D28: SMAJ400A, FOOTPRINTS:DIOM5026X229N, F.Cu at (180.4, 155.5)
- added D28: SMAJ400A, FOOTPRINTS:DIOM5026X229N, F.Cu at (180.4, 50.0)
- added D29: 5V6, Diode_SMD:D_SOD-123, F.Cu at (163.3, 75.3)
- added D29: 5V6, Diode_SMD:D_SOD-123, F.Cu at (163.3, 180.8)
- added D3: SMBJ14A, FOOTPRINTS:DIOM5436X261N, F.Cu at (78.5, 154.5)
- added D3: SMBJ14A, FOOTPRINTS:DIOM5436X261N, F.Cu at (78.5, 49.0)
- added D30: RS1MFP, Diode_SMD:D_SOD-123, F.Cu at (160.8, 75.3)
- added D30: RS1MFP, Diode_SMD:D_SOD-123, F.Cu at (160.8, 180.8)
- added D31: RS1MFP, Diode_SMD:D_SOD-123, F.Cu at (167.7, 62.1)
- added D31: RS1MFP, Diode_SMD:D_SOD-123, F.Cu at (167.7, 167.6)
- added D48: SMAJ400A, FOOTPRINTS:DIOM5026X229N, F.Cu at (174.1, 156.7)
- added D48: SMAJ400A, FOOTPRINTS:DIOM5026X229N, F.Cu at (174.1, 51.2)
- added D49: 5V6, Diode_SMD:D_SOD-123, F.Cu at (215.5, 59.6)
- added D49: 5V6, Diode_SMD:D_SOD-123, F.Cu at (215.5, 165.2)
- added D50: RS1MFP, Diode_SMD:D_SOD-123, F.Cu at (212.0, 62.0)
- added D50: RS1MFP, Diode_SMD:D_SOD-123, F.Cu at (212.0, 167.5)
- added D51: RS1MFP, Diode_SMD:D_SOD-123, F.Cu at (198.5, 159.0)
- added D51: RS1MFP, Diode_SMD:D_SOD-123, F.Cu at (198.5, 53.5)
- added D52: SMAJ400A, FOOTPRINTS:DIOM5026X229N, F.Cu at (197.0, 164.0)
- added D52: SMAJ400A, FOOTPRINTS:DIOM5026X229N, F.Cu at (197.0, 58.5)
- added D53: 5V6, Diode_SMD:D_SOD-123, F.Cu at (225.0, 69.5)
- added D53: 5V6, Diode_SMD:D_SOD-123, F.Cu at (225.0, 175.0)
- added D54: RS1MFP, Diode_SMD:D_SOD-123, F.Cu at (228.0, 69.5)
- added D54: RS1MFP, Diode_SMD:D_SOD-123, F.Cu at (228.0, 175.0)
- added D55: RS1MFP, Diode_SMD:D_SOD-123, F.Cu at (240.2, 48.5)
- added D55: RS1MFP, Diode_SMD:D_SOD-123, F.Cu at (240.2, 154.0)
- added D56: SMAJ400A, FOOTPRINTS:DIOM5026X229N, F.Cu at (236.5, 56.5)
- added D56: SMAJ400A, FOOTPRINTS:DIOM5026X229N, F.Cu at (236.5, 162.0)
- added D7: 5V6, Diode_SMD:D_SOD-123, F.Cu at (191.2, 164.0)
- added D7: 5V6, Diode_SMD:D_SOD-123, F.Cu at (191.2, 58.5)
- added F1: SF-3812TL400T-2, FOOTPRINTS:SF3812TL400T2, F.Cu at (53.9, 155.2)
- added F1: SF-3812TL400T-2, FOOTPRINTS:SF3812TL400T2, F.Cu at (53.9, 49.7)
- added G***: LOGO, CM4IO:ARP_Logo, F.Cu at (51.9, 134.1)
- added G***: LOGO, CM4IO:ARP_Logo, F.Cu at (51.9, 28.6)
- added H10: MountingHole_Pad, MountingHole:MountingHole_3.2mm_M3_DIN965_Pad_TopBottom, F.Cu at (73.5, 213.0)
- added H10: MountingHole_Pad, MountingHole:MountingHole_3.2mm_M3_DIN965_Pad_TopBottom, F.Cu at (73.5, 107.5)
- added H11: MountingHole_Pad, MountingHole:MountingHole_3.2mm_M3_DIN965_Pad_TopBottom, F.Cu at (191.5, 182.5)
- added H11: MountingHole_Pad, MountingHole:MountingHole_3.2mm_M3_DIN965_Pad_TopBottom, F.Cu at (191.5, 77.0)
- added H12: MountingHole_Pad, MountingHole:MountingHole_3.2mm_M3_DIN965_Pad_TopBottom, F.Cu at (58.3, 108.5)
- added H12: MountingHole_Pad, MountingHole:MountingHole_3.2mm_M3_DIN965_Pad_TopBottom, F.Cu at (58.3, 214.0)
- added H13: MountingHole_Pad, MountingHole:MountingHole_3.2mm_M3_DIN965_Pad_TopBottom, F.Cu at (179.0, 182.5)
- added H13: MountingHole_Pad, MountingHole:MountingHole_3.2mm_M3_DIN965_Pad_TopBottom, F.Cu at (179.0, 77.0)
- added H14: MountingHole_Pad, MountingHole:MountingHole_3.2mm_M3_DIN965_Pad_TopBottom, F.Cu at (88.0, 213.0)
- added H14: MountingHole_Pad, MountingHole:MountingHole_3.2mm_M3_DIN965_Pad_TopBottom, F.Cu at (88.0, 107.5)
- added H15: MountingHole_Pad, MountingHole:MountingHole_3.2mm_M3_DIN965_Pad_TopBottom, F.Cu at (203.5, 182.5)
- added H15: MountingHole_Pad, MountingHole:MountingHole_3.2mm_M3_DIN965_Pad_TopBottom, F.Cu at (203.5, 77.0)
- added H16: MountingHole_Pad, MountingHole:MountingHole_3.2mm_M3_DIN965_Pad_TopBottom, F.Cu at (103.0, 107.5)
- added H16: MountingHole_Pad, MountingHole:MountingHole_3.2mm_M3_DIN965_Pad_TopBottom, F.Cu at (103.0, 213.0)
- added H17: MountingHole_Pad, MountingHole:MountingHole_3.2mm_M3_DIN965_Pad_TopBottom, F.Cu at (217.0, 77.0)
- added H17: MountingHole_Pad, MountingHole:MountingHole_3.2mm_M3_DIN965_Pad_TopBottom, F.Cu at (217.0, 182.5)
- added H19: MountingHole_Pad, MountingHole:MountingHole_3.2mm_M3_DIN965_Pad_TopBottom, F.Cu at (239.8, 113.4)
- added H19: MountingHole_Pad, MountingHole:MountingHole_3.2mm_M3_DIN965_Pad_TopBottom, F.Cu at (239.8, 218.9)
- added H5: MountingHole_Pad, MountingHole:MountingHole_3.2mm_M3_DIN965_Pad_TopBottom, F.Cu at (119.0, 107.5)
- added H5: MountingHole_Pad, MountingHole:MountingHole_3.2mm_M3_DIN965_Pad_TopBottom, F.Cu at (119.0, 213.0)
- added H6: MountingHole_Pad, MountingHole:MountingHole_5.3mm_M5_DIN965_Pad_TopBottom, F.Cu at (244.9, 38.3)
- added H6: MountingHole_Pad, MountingHole:MountingHole_5.3mm_M5_DIN965_Pad_TopBottom, F.Cu at (244.9, 143.8)
- added H7: MountingHole_Pad, MountingHole:MountingHole_5.3mm_M5_DIN965_Pad_TopBottom, F.Cu at (244.9, 77.0)
- added H7: MountingHole_Pad, MountingHole:MountingHole_5.3mm_M5_DIN965_Pad_TopBottom, F.Cu at (244.9, 182.5)
- added H8: MountingHole_Pad, MountingHole:MountingHole_5.3mm_M5_DIN965_Pad_TopBottom, F.Cu at (51.7, 38.3)
- added H8: MountingHole_Pad, MountingHole:MountingHole_5.3mm_M5_DIN965_Pad_TopBottom, F.Cu at (51.7, 143.8)
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Routing:
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- added copper zone on F.Cu, net Board_0-+12V
- added copper zone on F.Cu, net Board_0-+12V_EXT
- added copper zone on F.Cu, net Board_0-+3V3
- added copper zone on In2.Cu, net Board_0-+3V3
- added copper zone on B.Cu, net Board_0-/Line1_RelayIN
- added copper zone on F.Cu, net Board_0-/Line1_RelayIN
- added copper zone on In1.Cu, net Board_0-/Line1_RelayIN
- added copper zone on In2.Cu, net Board_0-/Line1_RelayIN
- added copper zone on B.Cu, net Board_0-/Line2_RelayIN
- added copper zone on F.Cu, net Board_0-/Line2_RelayIN
- added copper zone on In1.Cu, net Board_0-/Line2_RelayIN
- added copper zone on In2.Cu, net Board_0-/Line2_RelayIN
- added copper zone on B.Cu, net Board_0-/Line3_RelayIN
- added copper zone on F.Cu, net Board_0-/Line3_RelayIN
- added copper zone on In1.Cu, net Board_0-/Line3_RelayIN
- added copper zone on In2.Cu, net Board_0-/Line3_RelayIN
- added copper zone on B.Cu, net Board_0-/Line_1
- added copper zone on F.Cu, net Board_0-/Line_1
- added copper zone on In1.Cu, net Board_0-/Line_1
- added copper zone on In2.Cu, net Board_0-/Line_1
- added copper zone on B.Cu, net Board_0-/Line_1_OUT
- added copper zone on F.Cu, net Board_0-/Line_1_OUT
- added copper zone on In1.Cu, net Board_0-/Line_1_OUT
- added copper zone on In2.Cu, net Board_0-/Line_1_OUT
- added copper zone on B.Cu, net Board_0-/Line_2
- added copper zone on F.Cu, net Board_0-/Line_2
- added copper zone on In1.Cu, net Board_0-/Line_2
- added copper zone on In2.Cu, net Board_0-/Line_2
- added copper zone on B.Cu, net Board_0-/Line_2_OUT
- added copper zone on F.Cu, net Board_0-/Line_2_OUT
- added copper zone on In1.Cu, net Board_0-/Line_2_OUT
- added copper zone on In2.Cu, net Board_0-/Line_2_OUT
- added copper zone on B.Cu, net Board_0-/Line_3
- added copper zone on F.Cu, net Board_0-/Line_3
- added copper zone on In1.Cu, net Board_0-/Line_3
- added copper zone on In2.Cu, net Board_0-/Line_3
- added copper zone on B.Cu, net Board_0-/Line_3_OUT
- added copper zone on F.Cu, net Board_0-/Line_3_OUT
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Other:
- board size 205 x 105.5 mm -> 219 x 225 mm
- board text added: "JLCJLCJLCJLC"
- board text added: "V-CUT"
- board text removed: "OUT"
